File: forager-pcb/forager-pcb.kicad_pcb (KiCad board)
At the start: 2 copper layers, 236.5 x 96.3 mm, 90 parts, among them J1 Conn_01x02_Pin, J2 Conn_01x02_Pin

Commit message: Re-grid Forager to 19x19 mm pitch; add Choc v2 hotswap footprint lib
Keys moved to 19x19 pitch (column stagger and thumb angle kept), traces,
vias, outline, zones remapped. Schematic switch footprints set to
marbastlib-xp-choc:SW_choc_v2_HS_CPG135001S30_1u.

Co-Authored-By: Claude Opus 5.5 <noreply@anthropic.com>
Parts:
- moved LCH1 4.47 mm to (-111.0, -30.0)
- moved LCH11 4.47 mm to (-111.0, 8.00)
- moved LU1 4.47 mm to (-111.5, -42.0)
- moved RCH15 4.47 mm to (111.0, 8.00)
- moved RCH5 4.47 mm to (111.0, -30.0)
- moved RU1 4.47 mm to (111.5, -42.0)
- moved LCH6 4.00 mm to (-111.0, -11.0)
- moved RCH10 4.00 mm to (111.0, -11.0)
- moved REF** 3.80 mm to (-96.5, -47.8)
- moved REF** 3.80 mm to (96.5, 14.8)
- moved REF** 3.80 mm to (-96.5, 14.8)
- moved REF** 3.80 mm to (96.5, -47.8)
- moved J1 3.75 mm to (-95.2, 8.00)
- moved J2 3.75 mm to (95.2, 8.00)
- moved LCH12 3.61 mm to (-92.0, 2.00)
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Routing:
- net /LROW3: track 159.1 -> 169.4 mm
- net /RCOL4: track 156.1 -> 165.7 mm
- net /LCOL4: track 153.3 -> 162.4 mm
- net /LROW1: track 136.9 -> 145.9 mm
- net /RCOL3: track 135.8 -> 143.5 mm
- net /RROW3: track 110.5 -> 118.1 mm
- net /LCOL3: track 133.6 -> 141.0 mm
- net /RROW2: track 113.4 -> 120.7 mm
- net /LROW2: track 84.9 -> 91.4 mm
- net /RCOL2: track 76.3 -> 81.8 mm
- net /LCOL2: track 97.2 -> 102.5 mm
- net LBAT: track 90.7 -> 95.7 mm
- net Net-(LD7-A): track 66.7 -> 71.6 mm
- net RBAT: track 83.9 -> 88.7 mm
- net Net-(LD1-A): track 66.0 -> 70.7 mm
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Other:
- board size 236.5 x 96.3 mm -> 244.5 x 101.8 mm

Commit message: Use post-less Choc v2 hotswap footprint (5.0mm centre stem) for all switches
New project lib forager.pretty with SW_choc_v2_HS_CPG135001S30_1u_nopost,
derived from marbastlib (side positioning post removed).

Co-Authored-By: Claude Opus 5.5 <noreply@anthropic.com>
Parts:
- LCH1, LCH10, LCH11, LCH12, LCH13, LCH14, LCH15, LCH16, LCH17, LCH2, LCH3, LCH4, LCH5, LCH6, LCH7, LCH8, LCH9, RCH1, RCH10, RCH11, RCH12, RCH13, RCH14, RCH15, RCH16, RCH17, RCH2, RCH3, RCH4, RCH5, RCH6, RCH7, RCH8, RCH9: footprint Custom:SW_choc_v1_HS_MBK -> forager:SW_choc_v2_HS_CPG135001S30_1u_nopost

Commit message: Reroute traces around Choc v2 5mm centre holes
45 trace chains locally rerouted (6 hop layers via 2 vias each), 3 GND
vias nudged, near-miss clearances fixed. DRC: 0 unconnected; remaining
errors are 2 XIAO pin-to-centre-hole and 5 XIAO GND thermal spokes.

Co-Authored-By: Claude Opus 5.5 <noreply@anthropic.com>
Routing:
- net /LCOL1: track 86.7 -> 91.1 mm
- net Net-(LD8-A): track 46.9 -> 51.2 mm
- net /LCOL2: track 102.5 -> 106.2 mm
- net Net-(LD1-A): track 70.7 -> 67.4 mm
- net RBAT: track 88.7 -> 85.9 mm, vias 0 -> 6
- net /RROW3: track 118.1 -> 120.6 mm, vias 0 -> 2
- net /RROW2: track 120.7 -> 118.6 mm
- net Net-(RD16-A): track 33.3 -> 35.0 mm
- net Net-(RD9-A): track 29.9 -> 29.1 mm
- net /LCOL3: track 141.0 -> 140.9 mm, vias 1 -> 5
