File: forager-pcb/forager-pcb.kicad_pcb (KiCad board)
At the start: 2 copper layers, 244.5 x 101.8 mm, 90 parts, among them J1 Conn_01x02_Pin, J2 Conn_01x02_Pin

Commit message: Move XIAOs 0.3mm up for centre-hole clearance; tie XIAO GND pads to fill
DRC: 0 errors, 0 unconnected.

Co-Authored-By: Claude Opus 5.5 <noreply@anthropic.com>
Parts:
- moved LU1 0.30 mm to (-111.5, -42.3)
- moved RU1 0.30 mm to (111.5, -42.3)
Routing:
- net RGND: track 0.00 -> 3.00 mm
Changed lines of the file:
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@@
 	(footprint "Custom:xiao-ble-smd-cutout"
 		(layer "B.Cu")
-		(at -111.5 -42 -90)
+		(at -111.5 -42.3 -90)
 		(property "Reference" "LU1"
 			(at -19.3989 11.28268 90)
@@
 		(sheetname "/")
 		(sheetfile "forager-pcb.kicad_sch")
-		(units
-			(unit
-				(name "A")
-				(pins "1" "2" "3" "4" "5" "6" "7" "15" "16" "19" "20" "21" "22" "17"
-					"18" "8" "9" "10" "11" "12" "13" "14"
-				)
-			)
-		)
 		(attr smd exclude_from_bom)
 		(duplicate_pad_numbers_are_jumpers no)
@@
 	(footprint "Custom:xiao-ble-smd-cutout"
 		(layer "B.Cu")
-		(at 111.5 -42 90)
+		(at 111.5 -42.3 90)
 		(property "Reference" "RU1"
 			(at -19.3989 11.28268 90)
@@
 		(sheetname "/")
 		(sheetfile "forager-pcb.kicad_sch")
-		(units
-			(unit
-				(name "A")
-				(pins "1" "2" "3" "4" "5" "6" "7" "15" "16" "19" "20" "21" "22" "17"
-					"18" "8" "9" "10" "11" "12" "13" "14"
-				)
-			)
-		)
 		(attr smd exclude_from_bom)
 		(duplicate_pad_numbers_are_jumpers no)
@@
 	)
 	(gr_circle
-		(center -111.810753 -46.451247)
-		(end -110.610753 -46.451247)
+		(center -111.810753 -46.751247)
+		(end -110.610753 -46.751247)
 		(stroke
 			(width 0.2)
@@
 	)
 	(gr_circle
-		(center 111.810753 -37.548753)
-		(end 113.010753 -37.548753)
+		(center 111.810753 -37.848753)
+		(end 113.010753 -37.848753)
 		(stroke
 			(width 0.2)
@@
 	(segment
 		(start 102.35 -51.15)
-		(end 103.88 -49.62)
+		(end 103.88 -49.92)
 		(width 0.2)
 		(layer "B.Cu")
@@
 	)
 	(segment
-		(start 119.12 -34.38)
+		(start 119.12 -34.68)
 		(end 119.12 -30.62)
 		(width 0.2)
@@
 	)
 	(segment
-		(start 116.58 -34.38)
+		(start 116.58 -34.68)
 		(end 116.58 -32.42)
 		(width 0.2)
@@
 	)
 	(segment
-		(start 114.04 -34.38)
+		(start 114.04 -34.68)
 		(end 114.04 -31.96)
 		(width 0.2)
@@
 	(segment
 		(start -103.76 -49.5)
-		(end -103.88 -49.62)
+		(end -103.88 -49.92)
 		(width 0.2)
 		(layer "B.Cu")
@@
 	(segment
 		(start 111.5 -47)
-		(end 111.5 -49.62)
+		(end 111.5 -49.92)
 		(width 0.2)
 		(layer "B.Cu")
@@
 	)
 	(segment
-		(start 108.96 -34.38)
+		(start 108.96 -34.68)
 		(end 108.3 -31.5)
 		(width 0.2)
@@
 		(net "Net-(RD15-A)")
 	)
+	(segment
+		(start 113.722 -37.855)
+		(end 113.591266 -36.360708)
+		(width 0.4)
+		(layer "F.Cu")
+		(net "RGND")
+	)
 	(via
 		(at 88.5 3.5)
@@
 	)
 	(segment
+		(start 116.58 -49.92)
+		(end 117.64066 -48.85934)
+		(width 0.4)
+		(layer "B.Cu")
+		(net "RGND")
+	)
+	(segment
 		(start -41.333333 -46.35)
 		(end -39.538889 -44.65)
@@
 		(polygon
 			(pts
-				(xy 96.5 -52) (xy 96.5 -32) (xy 104 -32) (xy 104 -52)
+				(xy 96.5 -52.3) (xy 96.5 -32.3) (xy 104 -32.3) (xy 104 -52.3)
 			)
 		)
@@
 		(polygon
 			(pts
-				(xy -96.5 -52) (xy -96.5 -32) (xy -104 -32) (xy -104 -52)
+				(xy -96.5 -52.3) (xy -96.5 -32.3) (xy -104 -32.3) (xy -104 -52.3)
 			)
 		)
