File: forager-pcb/forager-pcb.kicad_pcb (KiCad board)
At the start: 2 copper layers, 244.5 x 101.8 mm, 90 parts, among them J1 Conn_01x02_Pin, J2 Conn_01x02_Pin

Commit message: Silkscreen: Forager / Choc v2 / rev. 1.0
Co-Authored-By: Claude Opus 5.5 <noreply@anthropic.com>
Other:
- board text added: "Choc v2"
- board text added: "rev. 1.0"
- board text removed: "rev. 2"

Commit message: Add Alps SSSS811101 power switches (up = on) on outer edges
- New footprint forager:SW_SPDT_Alps_SSSS811101 (Alps land pattern) + simple 3D model
- Schematic: LSW1/RSW1 in series with battery; XIAO BAT+ on new LBAT_SW/RBAT_SW nets
  (POWER class). Battery on the top pin of each switch, so slider up = on on both halves.
- PCB: switches on bottom at outer edge below XIAO, slider overhanging edge;
  battery lines rerouted, RROW2/RROW3 moved inward around RSW1, 3 GND vias removed.
- DRC: 0 errors, 0 unconnected.

Co-Authored-By: Claude Opus 5.5 <noreply@anthropic.com>
Parts:
- added LSW1: SSSS811101, forager:SW_SPDT_Alps_SSSS811101, B.Cu at (-120.4, -16.8)
- added RSW1: SSSS811101, forager:SW_SPDT_Alps_SSSS811101, B.Cu at (120.4, -16.8)
Connections:
- LU1 pad 16: LBAT -> LBAT_SW
- RU1 pad 16: RBAT -> RBAT_SW
Routing:
- net LBAT_SW: track 0.00 -> 41.8 mm
- net RBAT_SW: track 0.00 -> 41.5 mm, vias 0 -> 2
- net RBAT: track 85.9 -> 48.4 mm, vias 6 -> 8
- net LBAT: track 95.7 -> 60.2 mm
- net /RROW3: track 120.9 -> 121.8 mm
- net /RROW2: track 118.9 -> 119.7 mm
- net LGND: vias 28 -> 25

Commit message: Add optional Panasonic EVQ-PUC02K reset buttons on outer edges
- New footprint forager:SW_Panasonic_EVQPUC02K (Panasonic land pattern, with boss) + simple 3D model
- Schematic: LRST1/RRST1 between XIAO RST (pin 21) and GND; marked optional
  (XIAO onboard reset still works)
- PCB: bottom side, outer edge below the power switch, push plate ~1 mm past edge;
  RST routed from XIAO, left battery trace rerouted, RGND fill stitched, RST silkscreen
- DRC: 0 errors, 0 unconnected; ERC unchanged from original

Co-Authored-By: Claude Opus 5.5 <noreply@anthropic.com>
Parts:
- added LRST1: EVQ-PUC02K (optional), forager:SW_Panasonic_EVQPUC02K, B.Cu at (-120.5, 3.50)
- added RRST1: EVQ-PUC02K (optional), forager:SW_Panasonic_EVQPUC02K, B.Cu at (120.5, 3.50)
Connections:
- LU1 pad 21: unconnected-(LU1-RST-Pad21) -> LRST
- RU1 pad 21: unconnected-(RU1-RST-Pad21) -> RRST
Routing:
- net LRST: track 0.00 -> 50.5 mm, vias 0 -> 2
- net RRST: track 0.00 -> 48.7 mm
- net RGND: vias 18 -> 20
Other:
- board text added: "RST"
