File: forager-pcb/forager-pcb.kicad_sch (KiCad schematic)
At the start: 76 parts, among them J1 Conn_01x02_Pin, J2 Conn_01x02_Pin

Commit message: Re-grid Forager to 19x19 mm pitch; add Choc v2 hotswap footprint lib
Keys moved to 19x19 pitch (column stagger and thumb angle kept), traces,
vias, outline, zones remapped. Schematic switch footprints set to
marbastlib-xp-choc:SW_choc_v2_HS_CPG135001S30_1u.

Co-Authored-By: Claude Opus 5.5 <noreply@anthropic.com>
Parts:
- LCH1, LCH10, LCH11, LCH12, LCH13, LCH14, LCH15, LCH16, LCH17, LCH2, LCH3, LCH4, LCH5, LCH6, LCH7, LCH8, LCH9, RCH1, RCH10, RCH11, RCH12, RCH13, RCH14, RCH15, RCH16, RCH17, RCH2, RCH3, RCH4, RCH5, RCH6, RCH7, RCH8, RCH9: footprint Custom:SW_choc_v1_HS_MBK -> marbastlib-xp-choc:SW_choc_v2_HS_CPG135001S30_1u
Changed lines of the file:
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@@
 			)
 		)
-		(property "Footprint" "Custom:SW_choc_v1_HS_MBK"
+		(property "Footprint" "marbastlib-xp-choc:SW_choc_v2_HS_CPG135001S30_1u"
 			(at 31.75 90.17 0)
 			(effects
@@
 			)
 		)
-		(property "Footprint" "Custom:SW_choc_v1_HS_MBK"
+		(property "Footprint" "marbastlib-xp-choc:SW_choc_v2_HS_CPG135001S30_1u"
 			(at 71.12 110.49 0)
 			(effects
@@
 			)
 		)
-		(property "Footprint" "Custom:SW_choc_v1_HS_MBK"
+		(property "Footprint" "marbastlib-xp-choc:SW_choc_v2_HS_CPG135001S30_1u"
 			(at 58.42 90.17 0)
 			(effects
@@
 			)
 		)
-		(property "Footprint" "Custom:SW_choc_v1_HS_MBK"
+		(property "Footprint" "marbastlib-xp-choc:SW_choc_v2_HS_CPG135001S30_1u"
 			(at 165.1 90.17 0)
 			(effects
@@
 			)
 		)
-		(property "Footprint" "Custom:SW_choc_v1_HS_MBK"
+		(property "Footprint" "marbastlib-xp-choc:SW_choc_v2_HS_CPG135001S30_1u"
 			(at 190.5 110.49 0)
 			(effects
@@
 			)
 		)
-		(property "Footprint" "Custom:SW_choc_v1_HS_MBK"
+		(property "Footprint" "marbastlib-xp-choc:SW_choc_v2_HS_CPG135001S30_1u"
 			(at 165.1 69.85 0)
 			(effects
@@
 			)
 		)
-		(property "Footprint" "Custom:SW_choc_v1_HS_MBK"
+		(property "Footprint" "marbastlib-xp-choc:SW_choc_v2_HS_CPG135001S30_1u"
 			(at 58.42 110.49 0)
 			(effects
@@
 			)
 		)
-		(property "Footprint" "Custom:SW_choc_v1_HS_MBK"
+		(property "Footprint" "marbastlib-xp-choc:SW_choc_v2_HS_CPG135001S30_1u"
 			(at 177.8 69.85 0)
 			(effects
@@
 			)
 		)
-		(property "Footprint" "Custom:SW_choc_v1_HS_MBK"
+		(property "Footprint" "marbastlib-xp-choc:SW_choc_v2_HS_CPG135001S30_1u"
 			(at 161.29 132.08 0)
 			(effects
@@
 			)
 		)
-		(property "Footprint" "Custom:SW_choc_v1_HS_MBK"
+		(property "Footprint" "marbastlib-xp-choc:SW_choc_v2_HS_CPG135001S30_1u"
 			(at 190.5 69.85 0)
 			(effects
@@
 			)
 		)
-		(property "Footprint" "Custom:SW_choc_v1_HS_MBK"
+		(property "Footprint" "marbastlib-xp-choc:SW_choc_v2_HS_CPG135001S30_1u"
 			(at 71.12 90.17 0)
 			(effects
@@
 			)
 		)
-		(property "Footprint" "Custom:SW_choc_v1_HS_MBK"
+		(property "Footprint" "marbastlib-xp-choc:SW_choc_v2_HS_CPG135001S30_1u"
 			(at 58.42 69.85 0)
 			(effects
@@
 			)
 		)
-		(property "Footprint" "Custom:SW_choc_v1_HS_MBK"
+		(property "Footprint" "marbastlib-xp-choc:SW_choc_v2_HS_CPG135001S30_1u"
 			(at 45.72 69.85 0)
 			(effects
@@
 			)
 		)
-		(property "Footprint" "Custom:SW_choc_v1_HS_MBK"
+		(property "Footprint" "marbastlib-xp-choc:SW_choc_v2_HS_CPG135001S30_1u"
 			(at 87.63 132.08 0)
 			(effects
@@
 			)
 		)
-		(property "Footprint" "Custom:SW_choc_v1_HS_MBK"
+		(property "Footprint" "marbastlib-xp-choc:SW_choc_v2_HS_CPG135001S30_1u"
 			(at 71.12 69.85 0)
 			(effects
@@
 			)
 		)
-		(property "Footprint" "Custom:SW_choc_v1_HS_MBK"
+		(property "Footprint" "marbastlib-xp-choc:SW_choc_v2_HS_CPG135001S30_1u"
 			(at 177.8 90.17 0)
 			(effects
@@
 			)
 		)
-		(property "Footprint" "Custom:SW_choc_v1_HS_MBK"
+		(property "Footprint" "marbastlib-xp-choc:SW_choc_v2_HS_CPG135001S30_1u"
 			(at 190.5 90.17 0)
 			(effects
@@
 			)
 		)
-		(property "Footprint" "Custom:SW_choc_v1_HS_MBK"
+		(property "Footprint" "marbastlib-xp-choc:SW_choc_v2_HS_CPG135001S30_1u"
 			(at 203.2 90.17 0)
 			(effects
@@
 			)
 		)
-		(property "Footprint" "Custom:SW_choc_v1_HS_MBK"
+		(property "Footprint" "marbastlib-xp-choc:SW_choc_v2_HS_CPG135001S30_1u"
 			(at 73.66 132.08 0)
 			(effects
@@
 			)
 		)
-		(property "Footprint" "Custom:SW_choc_v1_HS_MBK"
+		(property "Footprint" "marbastlib-xp-choc:SW_choc_v2_HS_CPG135001S30_1u"
 			(at 31.75 110.49 0)
 			(effects
@@
 			)
 		)
-		(property "Footprint" "Custom:SW_choc_v1_HS_MBK"
+		(property "Footprint" "marbastlib-xp-choc:SW_choc_v2_HS_CPG135001S30_1u"
 			(at 83.82 69.85 0)
 			(effects
@@
 			)
 		)
-		(property "Footprint" "Custom:SW_choc_v1_HS_MBK"
+		(property "Footprint" "marbastlib-xp-choc:SW_choc_v2_HS_CPG135001S30_1u"
 			(at 165.1 110.49 0)
 			(effects
@@
 			)
 		)
-		(property "Footprint" "Custom:SW_choc_v1_HS_MBK"
+		(property "Footprint" "marbastlib-xp-choc:SW_choc_v2_HS_CPG135001S30_1u"
 			(at 217.17 110.49 0)
 			(effects
@@
 			)
 		)
-		(property "Footprint" "Custom:SW_choc_v1_HS_MBK"
+		(property "Footprint" "marbastlib-xp-choc:SW_choc_v2_HS_CPG135001S30_1u"
 			(at 203.2 110.49 0)
 			(effects
@@
 			)
 		)
-		(property "Footprint" "Custom:SW_choc_v1_HS_MBK"
+		(property "Footprint" "marbastlib-xp-choc:SW_choc_v2_HS_CPG135001S30_1u"
 			(at 177.8 110.49 0)
 			(effects
@@
 			)
 		)
-		(property "Footprint" "Custom:SW_choc_v1_HS_MBK"
+		(property "Footprint" "marbastlib-xp-choc:SW_choc_v2_HS_CPG135001S30_1u"
 			(at 217.17 90.17 0)
 			(effects
@@
 			)
 		)
-		(property "Footprint" "Custom:SW_choc_v1_HS_MBK"
+		(property "Footprint" "marbastlib-xp-choc:SW_choc_v2_HS_CPG135001S30_1u"
 			(at 83.82 90.17 0)
 			(effects
@@
 			)
 		)
-		(property "Footprint" "Custom:SW_choc_v1_HS_MBK"
+		(property "Footprint" "marbastlib-xp-choc:SW_choc_v2_HS_CPG135001S30_1u"
 			(at 203.2 69.85 0)
 			(effects
@@
 			)
 		)
-		(property "Footprint" "Custom:SW_choc_v1_HS_MBK"
+		(property "Footprint" "marbastlib-xp-choc:SW_choc_v2_HS_CPG135001S30_1u"
 			(at 175.26 132.08 0)
 			(effects
@@
 			)
 		)
-		(property "Footprint" "Custom:SW_choc_v1_HS_MBK"
+		(property "Footprint" "marbastlib-xp-choc:SW_choc_v2_HS_CPG135001S30_1u"
 			(at 83.82 110.49 0)
 			(effects
@@
 			)
 		)
-		(property "Footprint" "Custom:SW_choc_v1_HS_MBK"
+		(property "Footprint" "marbastlib-xp-choc:SW_choc_v2_HS_CPG135001S30_1u"
 			(at 31.75 69.85 0)
 			(effects
@@
 			)
 		)
-		(property "Footprint" "Custom:SW_choc_v1_HS_MBK"
+		(property "Footprint" "marbastlib-xp-choc:SW_choc_v2_HS_CPG135001S30_1u"
 			(at 45.72 110.49 0)
 			(effects
@@
 			)
 		)
-		(property "Footprint" "Custom:SW_choc_v1_HS_MBK"
+		(property "Footprint" "marbastlib-xp-choc:SW_choc_v2_HS_CPG135001S30_1u"
 			(at 217.17 69.85 0)
 			(effects
@@
 			)
 		)
-		(property "Footprint" "Custom:SW_choc_v1_HS_MBK"
+		(property "Footprint" "marbastlib-xp-choc:SW_choc_v2_HS_CPG135001S30_1u"
 			(at 45.72 90.17 0)
 			(effects

Commit message: Use post-less Choc v2 hotswap footprint (5.0mm centre stem) for all switches
New project lib forager.pretty with SW_choc_v2_HS_CPG135001S30_1u_nopost,
derived from marbastlib (side positioning post removed).

Co-Authored-By: Claude Opus 5.5 <noreply@anthropic.com>
Parts:
- LCH1, LCH10, LCH11, LCH12, LCH13, LCH14, LCH15, LCH16, LCH17, LCH2, LCH3, LCH4, LCH5, LCH6, LCH7, LCH8, LCH9, RCH1, RCH10, RCH11, RCH12, RCH13, RCH14, RCH15, RCH16, RCH17, RCH2, RCH3, RCH4, RCH5, RCH6, RCH7, RCH8, RCH9: footprint marbastlib-xp-choc:SW_choc_v2_HS_CPG135001S30_1u -> forager:SW_choc_v2_HS_CPG135001S30_1u_nopost

Commit message: Add Alps SSSS811101 power switches (up = on) on outer edges
- New footprint forager:SW_SPDT_Alps_SSSS811101 (Alps land pattern) + simple 3D model
- Schematic: LSW1/RSW1 in series with battery; XIAO BAT+ on new LBAT_SW/RBAT_SW nets
  (POWER class). Battery on the top pin of each switch, so slider up = on on both halves.
- PCB: switches on bottom at outer edge below XIAO, slider overhanging edge;
  battery lines rerouted, RROW2/RROW3 moved inward around RSW1, 3 GND vias removed.
- DRC: 0 errors, 0 unconnected.

Co-Authored-By: Claude Opus 5.5 <noreply@anthropic.com>
Parts:
- added LSW1, RSW1: SSSS811101, forager:SW_SPDT_Alps_SSSS811101, symbol Switch:SW_SPDT
Connections:
- net LBAT: now also LSW1.3 (C); no longer LU1.16 (BAT+)
- net RBAT: now also RSW1.1 (A); no longer RU1.16 (BAT+)
- new net LBAT_SW: LSW1.2 (B), LU1.16 (BAT+)
- new net RBAT_SW: RSW1.2 (B), RU1.16 (BAT+)
- no-connect marks 16 -> 18

Commit message: Add optional Panasonic EVQ-PUC02K reset buttons on outer edges
- New footprint forager:SW_Panasonic_EVQPUC02K (Panasonic land pattern, with boss) + simple 3D model
- Schematic: LRST1/RRST1 between XIAO RST (pin 21) and GND; marked optional
  (XIAO onboard reset still works)
- PCB: bottom side, outer edge below the power switch, push plate ~1 mm past edge;
  RST routed from XIAO, left battery trace rerouted, RGND fill stitched, RST silkscreen
- DRC: 0 errors, 0 unconnected; ERC unchanged from original

Co-Authored-By: Claude Opus 5.5 <noreply@anthropic.com>
Parts:
- added LRST1, RRST1: EVQ-PUC02K (optional), forager:SW_Panasonic_EVQPUC02K, symbol Switch:SW_Push
Connections:
- net LGND: now also LRST1.2
- net RGND: now also RRST1.2
- net RRST: now reaches RU1.21 (RST)
- net RRST: now also RRST1.1
- net LRST: now reaches LU1.21 (RST)
- net LRST: now also LRST1.1
Other:
- note added: "OPTIONAL reset button - XIAO onboard reset still works"
Changed lines of the file:
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@@
 		)
 	)
+	(wire
+		(pts
+			(xy 96.52 54.61)
+			(xy 93.98 54.61)
+		)
+	)
+	(wire
+		(pts
+			(xy 106.68 54.61)
+			(xy 109.22 54.61)
+		)
+	)
+	(wire
+		(pts
+			(xy 46.99 16.51)
+			(xy 46.99 11.43)
+		)
+	)
+	(wire
+		(pts
+			(xy 232.41 54.61)
+			(xy 229.87 54.61)
+		)
+	)
+	(wire
+		(pts
+			(xy 242.57 54.61)
+			(xy 245.11 54.61)
+		)
+	)
+	(wire
+		(pts
+			(xy 182.88 16.51)
+			(xy 182.88 11.43)
+		)
+	)
 	(label "LROW0"
 		(at 20.32 36.83 0)
@@
 		)
 	)
+	(global_label "LRST"
+		(shape input)
+		(at 93.98 54.61 180)
+		(effects
+			(font
+				(size 1.27 1.27)
+			)
+			(justify right)
+		)
+	)
+	(global_label "LGND"
+		(shape input)
+		(at 109.22 54.61 0)
+		(effects
+			(font
+				(size 1.27 1.27)
+			)
+			(justify left)
+		)
+	)
+	(global_label "LRST"
+		(shape input)
+		(at 46.99 11.43 90)
+		(effects
+			(font
+				(size 1.27 1.27)
+			)
+			(justify left)
+		)
+	)
+	(global_label "RRST"
+		(shape input)
+		(at 229.87 54.61 180)
+		(effects
+			(font
+				(size 1.27 1.27)
+			)
+			(justify right)
+		)
+	)
+	(global_label "RGND"
+		(shape input)
+		(at 245.11 54.61 0)
+		(effects
+			(font
+				(size 1.27 1.27)
+			)
+			(justify left)
+		)
+	)
+	(global_label "RRST"
+		(shape input)
+		(at 182.88 11.43 90)
+		(effects
+			(font
+				(size 1.27 1.27)
+			)
+			(justify left)
+		)
+	)
+  (text "OPTIONAL reset button - XIAO onboard reset still works"
+    (at 88.9 62.23 0)
+    (effects (font (size 1.27 1.27)) (justify left bottom))
+  )
+  (text "OPTIONAL reset button - XIAO onboard reset still works"
+    (at 224.79 62.23 0)
+    (effects (font (size 1.27 1.27)) (justify left bottom))
+  )
 	(symbol
 		(lib_id "Device:D")
@@
 					(unit 1)
 				)
+			)
+		)
+	)
+	(symbol
+		(lib_id "Switch:SW_Push")
+		(at 101.6 54.61 0)
+		(unit 1)
+		(in_bom yes)
+		(on_board yes)
+		(dnp no)
+		(property "Reference" "LRST1"
+			(at 102.87 52.07 0)
+			(effects
+				(font
+					(size 1.27 1.27)
+				)
+				(justify left)
+			)
+		)
+		(property "Value" "EVQ-PUC02K (optional)"
+			(at 101.6 56.134 0)
+			(effects
+				(font
+					(size 1.27 1.27)
+				)
+			)
+		)
+		(property "Footprint" "forager:SW_Panasonic_EVQPUC02K"
+			(at 101.6 54.61 0)
+			(hide yes)
+			(effects
+				(font
+					(size 1.27 1.27)
+				)
+			)
+		)
+		(property "Datasheet" ""
+			(at 101.6 54.61 0)
+			(hide yes)
+			(effects
+				(font
+					(size 1.27 1.27)
+				)
+			)
+		)
+		(property "Description" "Push button switch, generic, two pins"
+			(at 101.6 54.61 0)
+			(hide yes)
+			(effects
+				(font
+					(size 1.27 1.27)
+				)
+			)
+		)
+		(instances
+			(project "forager-pcb"
+				(path "/25b48b1d-6487-48b5-9c33-d941f15e9f3f"
+					(reference "LRST1")
+					(unit 1)
+				)
+			)
+		)
+	)
+	(symbol
+		(lib_id "Switch:SW_Push")
+		(at 237.49 54.61 0)
+		(unit 1)
+		(in_bom yes)
+		(on_board yes)
+		(dnp no)
+		(property "Reference" "RRST1"
+			(at 238.76 52.07 0)
+			(effects
+				(font
+					(size 1.27 1.27)
+				)
+				(justify left)
+			)
+		)
+		(property "Value" "EVQ-PUC02K (optional)"
+			(at 237.49 56.134 0)
+			(effects
+				(font
+					(size 1.27 1.27)
+				)
+			)
+		)
+		(property "Footprint" "forager:SW_Panasonic_EVQPUC02K"
+			(at 237.49 54.61 0)
+			(hide yes)
+			(effects
+				(font
+					(size 1.27 1.27)
+				)
+			)
+		)
+		(property "Datasheet" ""
+			(at 237.49 54.61 0)
+			(hide yes)
+			(effects
+				(font
+					(size 1.27 1.27)
+				)
+			)
+		)
+		(property "Description" "Push button switch, generic, two pins"
+			(at 237.49 54.61 0)
+			(hide yes)
+			(effects
+				(font
+					(size 1.27 1.27)
+				)
+			)
+		)
+		(instances
+			(project "forager-pcb"
+				(path "/25b48b1d-6487-48b5-9c33-d941f15e9f3f"
+					(reference "RRST1")
+					(unit 1)
+				)

Commit message: Add 3x SK6812MINI-E status LEDs per half on the top inner edge
- Reverse-mount LEDs at 4.5 mm pitch near the inner standoff, chained
  from XIAO P0.05 via 330R; P-FET (AO3401A) high-side switch on 3V3,
  enabled active-low from P1.15 (left) / P1.11 (right), 100k gate
  pull-up, 1k gate resistor, 1uF bulk cap. 1206 hand-solder passives.
- Via-in-pad GND on the boxed-in LED VSS pads; B.Cu rule areas keep
  the back fill out of the LED pad row (fixes copper slivers).
- Re-route right RBAT_SW on F.Cu, move LD5 and re-route its anode,
  remove XIAO 3V3 no-connect flags.
- docs/led-indicators-handoff.md documents the design and open items.

DRC: 0 errors, 0 unconnected. ERC unchanged from baseline.

Co-Authored-By: Claude Opus 5.5 <noreply@anthropic.com>
Parts:
- added LC1, RC1: 1uF, Capacitor_SMD:C_1206_3216Metric_Pad1.33x1.80mm_HandSolder, symbol Device:C
- added LLED1, LLED2, LLED3, RLED1, RLED2, RLED3: SK6812MINI-E, LED_SMD:LED_SK6812MINI-E_3.2x2.8mm_P1.5mm_ReverseMount, symbol LED:SK6812MINI-E
- added LQ1, RQ1: AO3401A, Package_TO_SOT_SMD:SOT-23, symbol Transistor_FET:AO3401A
- added LR1, RR1: 100k, Resistor_SMD:R_1206_3216Metric_Pad1.30x1.75mm_HandSolder, symbol Device:R
- added LR2, RR2: 330, Resistor_SMD:R_1206_3216Metric_Pad1.30x1.75mm_HandSolder, symbol Device:R
- added LR3, RR3: 1k, Resistor_SMD:R_1206_3216Metric_Pad1.30x1.75mm_HandSolder, symbol Device:R
Connections:
- net LGND: now also LC1.2, LLED1.1 (VSS), LLED2.1 (VSS), LLED3.1 (VSS)
- net RGND: now also RC1.2, RLED1.1 (VSS), RLED2.1 (VSS), RLED3.1 (VSS)
- net R3V3: now reaches RU1.10 (3V3)
- net R3V3: now also RQ1.2 (S), RR1.1
- net RLED_DIN: now reaches RU1.6 (P0.05/5)
- net RLED_DIN: now also RR2.1
- net RLED_EN: now reaches RU1.7 (P1.11/6)
- net RLED_EN: now also RR3.1
- net L3V3: now reaches LU1.10 (3V3)
- net L3V3: now also LQ1.2 (S), LR1.1
- net LLED_EN: now reaches LU1.11 (P1.15/10)
- net LLED_EN: now also LR3.1
- net LLED_DIN: now reaches LU1.6 (P0.05/5)
- net LLED_DIN: now also LR2.1
- new net LLED_D1: LLED1.2 (DIN), LR2.2
- new net LLED_D2: LLED1.4 (DOUT), LLED2.2 (DIN)
- new net LLED_D3: LLED2.4 (DOUT), LLED3.2 (DIN)
- new net LLED_G: LQ1.1 (G), LR1.2, LR3.2
- new net LVLED: LC1.1, LLED1.3 (VDD), LLED2.3 (VDD), LLED3.3 (VDD), LQ1.3 (D)
- new net RLED_D1: RLED1.2 (DIN), RR2.2
- new net RLED_D2: RLED1.4 (DOUT), RLED2.2 (DIN)
- new net RLED_D3: RLED2.4 (DOUT), RLED3.2 (DIN)
- new net RLED_G: RQ1.1 (G), RR1.2, RR3.2
- new net RVLED: RC1.1, RLED1.3 (VDD), RLED2.3 (VDD), RLED3.3 (VDD), RQ1.3 (D)
